File: ESP32 Project/ESP32 Project.kicad_sch (KiCad schematic)
At the start: 1 part, among them J1 USB_C_Receptacle

Commit message: something more done
Parts:
- removed J1: USB_C_Receptacle, Connector_USB:USB_C_Receptacle_Amphenol_12401548E4-2A, symbol Connector:USB_C_Receptacle
- added J1: 2338792-1, 2338792-1:TE_2338792-1, symbol 2338792-1:2338792-1
- added J2: B2B-PH-SM4-TB, B2B-PH-SM4-TB:JST_B2B-PH-SM4-TB, symbol B2B-PH-SM4-TB:B2B-PH-SM4-TB
- added U1: MCP73871, Package_DFN_QFN:QFN-20-1EP_4x4mm_P0.5mm_EP2.5x2.5mm, symbol Battery_Management:MCP73871
- added VR1: LM1117MPX-3.3, LM1117MPX-3.3:VREG_LM1117MPX-3.3, symbol LM1117MPX-3.3:LM1117MPX-3.3
Connections:
- new net: J1.G1 (SHIELD), J1.G2 (SHIELD), J1.G3 (SHIELD), J1.G4 (SHIELD), J1.G5 (SHIELD), J1.G6 (SHIELD)
- new net: U1.1 (OUT), U1.20 (OUT)
- new net: U1.10 (V_{SS}), U1.11 (V_{SS}), U1.21 (V_{SS})
- new net: U1.14 (V_{BAT}), U1.15 (V_{BAT})
- new net: U1.18 (IN), U1.19 (IN)
- new net GND_A: J1.A1 (GND_A), J1.A12 (GND_A)
- new net GND_B: J1.B1 (GND_B), J1.B12 (GND_B)
- new net VBUS_A: J1.A4 (VBUS_A), J1.A9 (VBUS_A)
- new net VBUS_B: J1.B4 (VBUS_B), J1.B9 (VBUS_B)

Commit message: lipo charger + usb c connector + voltage regulator schema done
Parts:
- added C1: C, symbol Device:C
- added D1: LED_red, LED_SMD:LED_0805_2012Metric_Pad1.15x1.40mm_HandSolder, symbol Device:LED_Small
- added D2: LED_green, LED_SMD:LED_0805_2012Metric_Pad1.15x1.40mm_HandSolder, symbol Device:LED_Small
- added D3: LED_blue, LED_SMD:LED_0805_2012Metric_Pad1.15x1.40mm_HandSolder, symbol Device:LED_Small
- added F1, F2: 0ZCH0110AF2E, 0ZCH0110AF2E:FUSC3225X100N, symbol 0ZCH0110AF2E:0ZCH0110AF2E
- added R1: 10k, symbol Device:R
- added R2: 10K, symbol Device:R
- added R3, R4: 5k1, symbol Device:R
- added R5: 2k, symbol Device:R
- added R6: 20k, symbol Device:R
- added R7, R8, R9: 470, symbol Device:R
Connections:
- net GND_A is gone; now on net GND: J1.A1 (GND_A), J1.A12 (GND_A)
- net GND_B is gone; now on net GND: J1.B1 (GND_B), J1.B12 (GND_B)
- net VBUS_B: now also C1.1, F1.2
- net at J1.A5 (CC1): now also R4.2
- net at J1.B5 (CC2): now also R3.2
- net GND: now reaches J1.G1 (SHIELD), J1.G2 (SHIELD), J1.G3 (SHIELD), J1.G4 (SHIELD), J1.G5 (SHIELD), J1.G6 (SHIELD)
- net GND: now also C1.2, D1.2 (A), D2.2 (A), D3.2 (A), R1.2, R2.2, R3.1, R4.1, R5.1, R6.1
- net at U1.12 (PROG3): now also R6.2
- net at U1.13 (PROG1): now also R5.2
- net at U1.5 (THERM): now also R2.1
- net at U1.6 (~{PG}): now also R9.2
- net at U1.7 (STAT2): now also R7.2
- net at U1.8 (STAT1/~{LBO}): now also R8.2
- net at U1.9 (~{TE}): now also R1.1
- new net: D1.1 (K), R7.1
- new net: D2.1 (K), R8.1
- new net: D3.1 (K), R9.1
- no-connect marks 0 -> 8
Other:
- moved on the sheet: J2, U1

Commit message: schema saved
Parts:
- added C2, C5: 0.1u, symbol Device:C
- added C3, C4: 10u, symbol Device:C_Polarized
- added C6: 10u, symbol Device:C
- C1: value C -> 0.1u
Connections:
- net VBUS_B is gone; now on net VBUS_A: C1.1, F1.2, J1.B4 (VBUS_B), J1.B9 (VBUS_B)
- net GND: now also U1.10 (V_{SS}), U1.11 (V_{SS}), U1.21 (V_{SS}), VR1.1 (GND), C2.2, C3.2, C4.2, C5.2, C6.2; no longer D1.2 (A), D2.2 (A), D3.2 (A)
- net 5volt usb: now reaches F1.1
- net 5volt usb: now also D1.2 (A), D2.2 (A), D3.2 (A), U1.18 (IN), U1.19 (IN), U1.2 (VPCC), C6.1
- net +3.3V: now reaches VR1.2 (VOUT_2)
- net +3.3V: now also VR1.4 (VOUT_4), C4.1, C5.1
- net +5Volt: now reaches VR1.3 (VIN)
- net +5Volt: now also U1.1 (OUT), U1.20 (OUT), C2.1, C3.1
- net USB-DP: now reaches J1.A6 (DP1)
- net USB-DP: now also J1.B6 (DP2)
- net USB-DN: now reaches J1.A7 (DN1)
- net USB-DN: now also J1.B7 (DN2)
- net Vbat: now reaches U1.14 (V_{BAT}), U1.15 (V_{BAT})
- net Vbat: now also U1.16 (V_{BAT_SENSE})
- no-connect marks 8 -> 10
Other:
- note added: "LiPo batt Charger"
- note added: "USB_C Connector"
- moved on the sheet: C1, F1, F2, J1, R3, R4
