File: ESP32 Project/ESP32 Project.kicad_sch (KiCad schematic)
At the start: 25 parts, among them J1 2338792-1, J2 B2B-PH-SM4-TB, U1 MCP73871

Commit message: most of the schema is done , esp32 page is done
Other:
- sheet Esp32-C2-02 ports: added USB-DN, USB-DP, VBUS; removed none
Changed lines of the file:
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@@
 		)
 	)
+	(label "USB-DP"
+		(at 208.28 114.3 0)
+		(effects
+			(font
+				(size 1.27 1.27)
+			)
+			(justify left bottom)
+		)
+	)
+	(label "USB-DN"
+		(at 208.28 118.11 0)
+		(effects
+			(font
+				(size 1.27 1.27)
+			)
+			(justify left bottom)
+		)
+	)
 	(label "Charging power good"
 		(at 189.23 40.64 90)
@@
 		)
 	)
+	(label "VBUS"
+		(at 208.28 121.92 0)
+		(effects
+			(font
+				(size 1.27 1.27)
+			)
+			(justify left bottom)
+		)
+	)
 	(label "USB-DP"
 		(at 76.2 45.72 0)
@@
 	)
 	(sheet
-		(at 141.605 107.95)
+		(at 164.465 105.41)
 		(size 43.815 49.53)
 		(exclude_from_sim no)
@@
 			(width 0.1524)
 			(type solid)
+			(color 57 78 255 1)
 		)
 		(fill
-			(color 0 0 0 0)
+			(color 133 255 255 1)
 		)
 		(property "Sheetname" "Esp32-C2-02"
-			(at 141.605 107.2384 0)
+			(at 164.465 104.6984 0)
 			(show_name no)
 			(do_not_autoplace no)
@@
 		)
 		(property "Sheetfile" "esp32-c3-02.kicad_sch"
-			(at 141.605 158.0646 0)
+			(at 164.465 155.5246 0)
 			(show_name no)
 			(do_not_autoplace no)
@@
 			)
 		)
+		(pin "USB-DP" input
+			(at 208.28 114.3 0)
+			(effects
+				(font
+					(size 1.27 1.27)
+				)
+				(justify right)
+			)
+		)
+		(pin "USB-DN" input
+			(at 208.28 118.11 0)
+			(effects
+				(font
+					(size 1.27 1.27)
+				)
+				(justify right)
+			)
+		)
+		(pin "VBUS" input
+			(at 208.28 121.92 0)
+			(effects
+				(font
+					(size 1.27 1.27)
+				)
+				(justify right)
+			)
+		)

Commit message: schema is done
Parts:
- C1, C2, C5: footprint (none) -> Capacitor_SMD:C_0805_2012Metric
- C3, C4: footprint (none) -> Capacitor_SMD:CP_Elec_4x3
- C6: value 10u -> 1u; footprint (none) -> Capacitor_SMD:C_0805_2012Metric
- R1, R10, R2, R3, R4, R5, R6, R7, R8, R9: footprint (none) -> Resistor_SMD:R_0805_2012Metric
Connections:
- net GND: now also U1.3 (SEL)

Commit message: something done lmao
Parts:
- C3, C4: footprint Capacitor_SMD:CP_Elec_4x3 -> Capacitor_SMD:C_Elec_5x5.4
Changed lines of the file:
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@@
 			)
 		)
-		(property "Footprint" "Capacitor_SMD:CP_Elec_4x3"
+		(property "Footprint" "Capacitor_SMD:C_Elec_5x5.4"
 			(at 82.8548 138.43 0)
 			(hide yes)
@@
 			)
 		)
-		(property "Footprint" "Capacitor_SMD:CP_Elec_4x3"
+		(property "Footprint" "Capacitor_SMD:C_Elec_5x5.4"
 			(at 31.4452 142.24 0)
 			(hide yes)

Commit message: pcb ont he way tomoroow
Parts:
- C3, C4: footprint Capacitor_SMD:C_Elec_5x5.4 -> Capacitor_Tantalum_SMD:CP_EIA-6032-28_Kemet-C
Changed lines of the file:
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@@
 			)
 		)
-		(property "Footprint" "Capacitor_SMD:C_Elec_5x5.4"
+		(property "Footprint" "Capacitor_Tantalum_SMD:CP_EIA-6032-28_Kemet-C"
 			(at 82.8548 138.43 0)
 			(hide yes)
@@
 			)
 		)
-		(property "Footprint" "Capacitor_SMD:C_Elec_5x5.4"
+		(property "Footprint" "Capacitor_Tantalum_SMD:CP_EIA-6032-28_Kemet-C"
 			(at 31.4452 142.24 0)
 			(hide yes)

Commit message: pcb done and some 3d models aadd
Parts:
- C3, C4: footprint Capacitor_Tantalum_SMD:CP_EIA-6032-28_Kemet-C -> Capacitor_Tantalum_SMD:CP_EIA-3216-12_Kemet-S
Changed lines of the file:
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@@
 			)
 		)
-		(property "Footprint" "Capacitor_Tantalum_SMD:CP_EIA-6032-28_Kemet-C"
+		(property "Footprint" "Capacitor_Tantalum_SMD:CP_EIA-3216-12_Kemet-S"
 			(at 82.8548 138.43 0)
 			(hide yes)
@@
 			)
 		)
-		(property "Footprint" "Capacitor_Tantalum_SMD:CP_EIA-6032-28_Kemet-C"
+		(property "Footprint" "Capacitor_Tantalum_SMD:CP_EIA-3216-12_Kemet-S"
 			(at 31.4452 142.24 0)
 			(hide yes)
