File: ESP32 Project/untitled.kicad_sch (KiCad schematic)
At the start: 0 parts

Commit message: we are at edge of work , almost complete and now going for the pcb design and routign
Parts:
- added J4: Conn_01x04_Pin, symbol Connector:Conn_01x04_Pin
- added J5: Conn_01x05_Pin, symbol Connector:Conn_01x05_Pin
- added Q2, Q3: BC817, Package_TO_SOT_SMD:SOT-23, symbol Transistor_BJT:BC817
- added R33, R34: 10k, symbol Device:R
- added S1, S2: USLPT2819DT2TR, USLPT2819DT2TR:SW_USLPT2819DT2TR, symbol USLPT2819DT2TR:USLPT2819DT2TR
Connections:
- new net: Q2.1 (B), R33.2
- new net: Q3.1 (B), R34.2
- new net +3.3V: J4.1 (Pin_1), J5.5 (Pin_5)
- new net DTR: Q3.3 (C), R33.1
- new net EN: Q2.3 (C)
- new net GND: J4.4 (Pin_4), J5.1 (Pin_1)
- new net GPIO18: J5.3 (Pin_3)
- new net GPIO8: J5.2 (Pin_2)
- new net GPIO9: J5.4 (Pin_4)
- new net IO0 / BOOT: Q3.2 (E)
- new net RTS: Q2.2 (E), R34.1
- new net SCL: J4.3 (Pin_3)
- new net SDA: J4.2 (Pin_2)
Other:
- note added: "OLED display connector I2C"
- title: (none) -> GPIO and I2C + BOOOT AND EN

Commit message: schema is done
Parts:
- added C21, C22: 0.1u, Capacitor_SMD:C_0805_2012Metric, symbol Device:C
- added R35: 10k, Resistor_SMD:R_0805_2012Metric, symbol Device:R
- J4: footprint (none) -> Connector_PinHeader_2.54mm:PinHeader_1x04_P2.54mm_Vertical
- J5: footprint (none) -> Connector_PinHeader_2.54mm:PinHeader_1x05_P2.54mm_Vertical
- R33, R34: footprint (none) -> Resistor_SMD:R_0805_2012Metric
- S1: value USLPT2819DT2TR -> USLPT2819DT2TR (BOOT)
- S2: value USLPT2819DT2TR -> USLPT2819DT2TR (RESET)
Connections:
- net +3.3V: now also R35.2
- net EN: now also S2.3, S2.4, C22.1, R35.1
- net GND: now also S1.1, S1.2, S2.1, S2.2, C21.2, C22.2
- net IO0 / BOOT: now also S1.3, S1.4, C21.1
- net GPIO9 renamed GPIO19
Other:
- note added: "Breakout of remaining pins"
- note added: "RESET and BOOT Buttons"
- moved on the sheet: J5, Q2, Q3, R33, R34, S1, S2
