File: ESP32 Project/sensors.kicad_sch (KiCad schematic)
At the start: 0 parts

Commit message: restart
Parts:
- added U6: BME280, Package_LGA:Bosch_LGA-8_2.5x2.5mm_P0.65mm_ClockwisePinNumbering, symbol Sensor:BME280
Changed lines of the file:
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@@
 	(generator_version "10.0")
 	(paper "A4")
+	(symbol
+		(lib_id "Sensor:BME280")
+		(at 44.45 45.72 0)
+		(unit 1)
+		(body_style 1)
+		(exclude_from_sim no)
+		(in_bom yes)
+		(on_board yes)
+		(in_pos_files yes)
+		(dnp no)
+		(fields_autoplaced yes)
+		(property "Reference" "U6"
+			(at 33.02 44.4499 0)
+			(show_name no)
+			(do_not_autoplace no)
+			(effects
+				(font
+					(size 1.27 1.27)
+				)
+				(justify right)
+			)
+		)
+		(property "Value" "BME280"
+			(at 33.02 46.9899 0)
+			(show_name no)
+			(do_not_autoplace no)
+			(effects
+				(font
+					(size 1.27 1.27)
+				)
+				(justify right)
+			)
+		)
+		(property "Footprint" "Package_LGA:Bosch_LGA-8_2.5x2.5mm_P0.65mm_ClockwisePinNumbering"
+			(at 82.55 57.15 0)
+			(hide yes)
+			(show_name no)
+			(do_not_autoplace no)
+			(effects
+				(font
+					(size 1.27 1.27)
+				)
+			)
+		)
+		(property "Datasheet" "https://www.bosch-sensortec.com/media/boschsensortec/downloads/datasheets/bst-bme280-ds002.pdf"
+			(at 44.45 50.8 0)
+			(hide yes)
+			(show_name no)
+			(do_not_autoplace no)
+			(effects
+				(font
+					(size 1.27 1.27)
+				)
+			)
+		)
+		(property "Description" "3-in-1 sensor, humidity, pressure, temperature, I2C and SPI interface, 1.71-3.6V, LGA-8"
+			(at 44.45 45.72 0)
+			(hide yes)
+			(show_name no)
+			(do_not_autoplace no)
+			(effects
+				(font
+					(size 1.27 1.27)
+				)
+			)
+		)
+		(pin "7"
+		)
+		(pin "1"
+		)
+		(pin "8"
+		)
+		(pin "3"
+		)
+		(pin "4"
+		)
+		(pin "5"
+		)
+		(pin "2"
+		)
+		(pin "6"
+		)
+		(instances
+			(project "ESP32 Project"
+				(path "/52b8cc89-874f-4cef-9400-6a059fb6c311/6085c309-5041-4ae1-96f0-edf60409793b/03b1f1e9-8a18-4af6-9122-b075f5380c8d"
+					(reference "U6")
+					(unit 1)
+				)
+			)
+		)
+	)
 )

Commit message: little bit of work done like bm280
Parts:
- added C15, C16: 0.1u, symbol Device:C
- added MK1: CMC-5042PF-AC, CMC-5042PF-AC:CUI_CMC-5042PF-AC, symbol CMC-5042PF-AC:CMC-5042PF-AC
- added Q1: TEMT6000X01, TEMT6000X01:TRANS_TEMT6000X01, symbol TEMT6000X01:TEMT6000X01
- added R24, R25: 4k7, symbol Device:R
- added U7: MAX4466EXK, MAX4466EXK:SOT65P210X110-5N, symbol MAX4466EXK:MAX4466EXK
Connections:
- net GND: now reaches U6.1 (GND)
- net GND: now also U6.5 (SDO), U6.7 (GND), C15.1, C16.1
- net +3.3V: now reaches U6.2 (CSB)
- net +3.3V: now also U6.6 (VDDIO), U6.8 (VDD), C15.2, C16.2, R24.1, R25.1
- net SDA: now reaches U6.3 (SDI)
- net SDA: now also R25.2
- net SCL: now reaches U6.4 (SCK)
- net SCL: now also R24.2
Other:
- note added: "BME 280 3 in 1 , humidity , temperature and presure"
- moved on the sheet: U6

Commit message: we are at edge of work , almost complete and now going for the pcb design and routign
Parts:
- removed C16: 0.1u, symbol Device:C
- added C18, C21: 0.1uf, symbol Device:C
- added C19: 1u, symbol Device:C
- added C20: 0.01uf, symbol Device:C
- added C20: 100pf, symbol Device:C
- added R23, R27: 10k, symbol Device:R
- added R28, R29: 1M, symbol Device:R
- added R30, R31: 2k, symbol Device:R
- added R31: 100k, symbol Device:R
Connections:
- net +3.3V: now also U7.5 (VCC), C18.2, R23.1, R29.2, R31.2
- net GND: now also MK1.GND, Q1.1, U7.2 (GND), C18.1, C19.2, C21.2, R28.1
- net at MK1.OUT: now also C20.2, R30.1
- net at U7.1 (IN+): now also C20.1, R28.2, R29.1
- net at U7.3 (IN-): now also C20.2, R27.2, R31.1
- net Mic_OUT: now reaches U7.4 (OUT)
- net Mic_OUT: now also C20.1, R31.2
- net PHOTO C: now reaches Q1.3
- net PHOTO C: now also R23.2
- new net: C21.1, R30.2, R31.1
- new net: C19.1, R27.1
Other:
- note added: "Microphone + amplifier"
- note added: "PHOTO sensor"
- moved on the sheet: MK1, Q1, U7

Commit message: schema is done
Parts:
- C15, C18, C19, C20: footprint (none) -> Capacitor_SMD:C_0805_2012Metric
- C24: renamed from C20; footprint (none) -> Capacitor_SMD:C_0805_2012Metric
- C25: renamed from C21; footprint (none) -> Capacitor_SMD:C_0805_2012Metric
- R23, R24, R25, R27, R28, R29, R30, R31: footprint (none) -> Resistor_SMD:R_0805_2012Metric
- R32: renamed from R31; footprint (none) -> Resistor_SMD:R_0805_2012Metric
Changed lines of the file:
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@@
 		(in_pos_files yes)
 		(dnp no)
-		(property "Reference" "R31"
+		(property "Reference" "R32"
 			(at 163.83 30.4801 0)
 			(show_name no)
@@
 			)
 		)
-		(property "Footprint" ""
+		(property "Footprint" "Resistor_SMD:R_0805_2012Metric"
 			(at 168.148 29.21 90)
 			(hide yes)
@@
 			(project "ESP32 Project"
 				(path "/52b8cc89-874f-4cef-9400-6a059fb6c311/6085c309-5041-4ae1-96f0-edf60409793b/03b1f1e9-8a18-4af6-9122-b075f5380c8d"
-					(reference "R31")
+					(reference "R32")
 					(unit 1)
 				)
@@
 			)
 		)
-		(property "Footprint" ""
+		(property "Footprint" "Resistor_SMD:R_0805_2012Metric"
 			(at 36.322 50.8 90)
 			(hide yes)
@@
 			)
 		)
-		(property "Footprint" ""
+		(property "Footprint" "Resistor_SMD:R_0805_2012Metric"
 			(at 196.088 58.42 90)
 			(hide yes)
@@
 			)
 		)
-		(property "Footprint" ""
+		(property "Footprint" "Resistor_SMD:R_0805_2012Metric"
 			(at 49.022 120.65 90)
 			(hide yes)
@@
 			)
 		)
-		(property "Footprint" ""
+		(property "Footprint" "Resistor_SMD:R_0805_2012Metric"
 			(at 26.162 50.8 90)
 			(hide yes)
@@
 			)
 		)
-		(property "Footprint" ""
+		(property "Footprint" "Resistor_SMD:R_0805_2012Metric"
 			(at 211.328 66.04 90)
 			(hide yes)
@@
 		(dnp no)
 		(fields_autoplaced yes)
-		(property "Reference" "C21"
+		(property "Reference" "C25"
 			(at 153.67 29.21 90)
 			(show_name no)
@@
 			)
 		)
-		(property "Footprint" ""
+		(property "Footprint" "Capacitor_SMD:C_0805_2012Metric"
 			(at 149.86 37.7952 0)
 			(hide yes)
@@
 			(project "ESP32 Project"
 				(path "/52b8cc89-874f-4cef-9400-6a059fb6c311/6085c309-5041-4ae1-96f0-edf60409793b/03b1f1e9-8a18-4af6-9122-b075f5380c8d"
-					(reference "C21")
+					(reference "C25")
 					(unit 1)
 				)
@@
 			)
 		)
-		(property "Footprint" ""
+		(property "Footprint" "Resistor_SMD:R_0805_2012Metric"
 			(at 168.148 43.18 90)
 			(hide yes)
@@
 			)
 		)
-		(property "Footprint" ""
+		(property "Footprint" "Capacitor_SMD:C_0805_2012Metric"
 			(at 267.0048 52.07 0)
 			(hide yes)
@@
 			)
 		)
-		(property "Footprint" ""
+		(property "Footprint" "Resistor_SMD:R_0805_2012Metric"
 			(at 196.088 43.18 90)
 			(hide yes)
@@
 			)
 		)
-		(property "Footprint" ""
+		(property "Footprint" "Resistor_SMD:R_0805_2012Metric"
 			(at 247.65 74.168 90)
 			(hide yes)
@@
 		(dnp no)
 		(fields_autoplaced yes)
-		(property "Reference" "C20"
+		(property "Reference" "C24"
 			(at 180.34 43.18 90)
 			(show_name no)
@@
 			)
 		)
-		(property "Footprint" ""
+		(property "Footprint" "Capacitor_SMD:C_0805_2012Metric"
 			(at 176.53 51.7652 0)
 			(hide yes)
@@
 			)
 		)
+		(property "Purpose" ""
+			(at 180.34 50.8 0)
+			(show_name no)
+			(do_not_autoplace no)
+			(effects
+				(font
+					(size 1.27 1.27)
+				)
+			)
+		)
 		(pin "1"
 		)
@@
 			(project "ESP32 Project"
 				(path "/52b8cc89-874f-4cef-9400-6a059fb6c311/6085c309-5041-4ae1-96f0-edf60409793b/03b1f1e9-8a18-4af6-9122-b075f5380c8d"
-					(reference "C20")
+					(reference "C24")
 					(unit 1)
 				)
@@
 			)
 		)
-		(property "Footprint" ""
+		(property "Footprint" "Capacitor_SMD:C_0805_2012Metric"
 			(at 65.0748 76.2 0)
 			(hide yes)
@@
 			)
 		)
-		(property "Footprint" ""
+		(property "Footprint" "Capacitor_SMD:C_0805_2012Metric"
 			(at 210.5152 83.82 0)
 			(hide yes)
@@
 			)
 		)
-		(property "Footprint" ""
+		(property "Footprint" "Capacitor_SMD:C_0805_2012Metric"
 			(at 243.84 84.7852 0)
 			(hide yes)

Commit message: pcb ont he way tomoroow
Other:
- moved on the sheet: Q1, R23
Changed lines of the file:
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@@
 	)
 	(junction
-		(at 50.8 139.7)
+		(at 48.26 140.97)
 		(diameter 0)
 		(color 0 0 0 0)
@@
 	(wire
 		(pts
-			(xy 40.64 139.7) (xy 50.8 139.7)
+			(xy 38.1 140.97) (xy 48.26 140.97)
 		)
 		(stroke
@@
 	(wire
 		(pts
-			(xy 50.8 113.03) (xy 50.8 116.84)
+			(xy 48.26 114.3) (xy 48.26 118.11)
 		)
 		(stroke
@@
 	(wire
 		(pts
-			(xy 25.4 139.7) (xy 25.4 143.51)
+			(xy 22.86 140.97) (xy 22.86 144.78)
 		)
 		(stroke
@@
 	(wire
 		(pts
-			(xy 50.8 124.46) (xy 50.8 139.7)
+			(xy 48.26 125.73) (xy 48.26 140.97)
 		)
 		(stroke
@@
 	(wire
 		(pts
-			(xy 50.8 139.7) (xy 63.5 139.7)
+			(xy 48.26 140.97) (xy 60.96 140.97)
 		)
 		(stroke
@@
 	(wire
 		(pts
-			(xy 30.48 139.7) (xy 25.4 139.7)
+			(xy 27.94 140.97) (xy 22.86 140.97)
 		)
 		(stroke
@@
 	(hierarchical_label "PHOTO C"
 		(shape output)
-		(at 63.5 139.7 0)
+		(at 60.96 140.97 0)
 		(effects
 			(font
@@
 	(symbol
 		(lib_id "power:GND")
-		(at 25.4 143.51 0)
+		(at 22.86 144.78 0)
 		(unit 1)
 		(body_style 1)
@@
 		(fields_autoplaced yes)
 		(property "Reference" "#PWR035"
-			(at 25.4 149.86 0)
+			(at 22.86 151.13 0)
 			(hide yes)
 			(show_name no)
@@
 		)
 		(property "Value" "GND"
-			(at 25.4 148.59 0)
+			(at 22.86 149.86 0)
 			(show_name no)
 			(do_not_autoplace no)
@@
 		)
 		(property "Footprint" ""
-			(at 25.4 143.51 0)
+			(at 22.86 144.78 0)
 			(hide yes)
 			(show_name no)
@@
 		)
 		(property "Datasheet" ""
-			(at 25.4 143.51 0)
+			(at 22.86 144.78 0)
 			(hide yes)
 			(show_name no)
@@
 		)
 		(property "Description" "Power symbol creates a global label with name \"GND\" , ground"
-			(at 25.4 143.51 0)
+			(at 22.86 144.78 0)
 			(hide yes)
 			(show_name no)
@@
 	(symbol
 		(lib_id "Device:R")
-		(at 50.8 120.65 0)
+		(at 48.26 121.92 0)
 		(unit 1)
 		(body_style 1)
@@
 		(fields_autoplaced yes)
 		(property "Reference" "R23"
-			(at 53.34 119.3799 0)
+			(at 50.8 120.6499 0)
 			(show_name no)
 			(do_not_autoplace no)
@@
 		)
 		(property "Value" "10k"
-			(at 53.34 121.9199 0)
+			(at 50.8 123.1899 0)
 			(show_name no)
 			(do_not_autoplace no)
@@
 		)
 		(property "Footprint" "Resistor_SMD:R_0805_2012Metric"
-			(at 49.022 120.65 90)
+			(at 46.482 121.92 90)
 			(hide yes)
 			(show_name no)
@@
 		)
 		(property "Datasheet" ""
-			(at 50.8 120.65 0)
+			(at 48.26 121.92 0)
 			(hide yes)
 			(show_name no)
@@
 		)
 		(property "Description" "Resistor"
-			(at 50.8 120.65 0)
+			(at 48.26 121.92 0)
 			(hide yes)
 			(show_name no)
@@
 		)
 		(property "Purpose" ""
-			(at 50.8 120.65 0)
+			(at 48.26 121.92 0)
 			(show_name no)
 			(do_not_autoplace no)
@@
 	(symbol
 		(lib_id "power:+3.3V")
-		(at 50.8 113.03 0)
+		(at 48.26 114.3 0)
 		(unit 1)
 		(body_style 1)
@@
 		(fields_autoplaced yes)
 		(property "Reference" "#PWR036"
-			(at 50.8 116.84 0)
+			(at 48.26 118.11 0)
 			(hide yes)
 			(show_name no)
@@
 		)
 		(property "Value" "+3.3V"
-			(at 50.8 107.95 0)
+			(at 48.26 109.22 0)
 			(show_name no)
 			(do_not_autoplace no)
@@
 		)
 		(property "Footprint" ""
-			(at 50.8 113.03 0)
+			(at 48.26 114.3 0)
 			(hide yes)
 			(show_name no)
@@
 		)
 		(property "Datasheet" ""
-			(at 50.8 113.03 0)
+			(at 48.26 114.3 0)
 			(hide yes)
 			(show_name no)
@@
 		)
 		(property "Description" "Power symbol creates a global label with name \"+3.3V\""
-			(at 50.8 113.03 0)
+			(at 48.26 114.3 0)
 			(hide yes)
 			(show_name no)
@@
 	(symbol
 		(lib_id "TEMT6000X01:TEMT6000X01")
-		(at 35.56 137.16 270)
+		(at 33.02 138.43 270)
 		(unit 1)
 		(body_style 1)
@@
 		(fields_autoplaced yes)
 		(property "Reference" "Q1"
-			(at 35.5854 128.27 90)
+			(at 33.0454 129.54 90)
 			(show_name no)
 			(do_not_autoplace no)
@@
 		)
 		(property "Value" "TEMT6000X01"
-			(at 35.5854 130.81 90)
+			(at 33.0454 132.08 90)
 			(show_name no)
 			(do_not_autoplace no)
@@
 		)
 		(property "Footprint" "TEMT6000X01:TRANS_TEMT6000X01"
-			(at 35.56 137.16 0)
+			(at 33.02 138.43 0)
 			(hide yes)
 			(show_name no)
@@
 		)
 		(property "Datasheet" ""
-			(at 35.56 137.16 0)
+			(at 33.02 138.43 0)
 			(hide yes)
 			(show_name no)
@@
 		)
 		(property "Description" "Phototransistors 570nm Top View 1206 (3216 Metric)"
-			(at 35.56 137.16 0)
+			(at 33.02 138.43 0)
 			(hide yes)
 			(show_name no)
@@
 		)
 		(property "MF" "Vishay Semiconductor"
-			(at 35.56 137.16 0)
+			(at 33.02 138.43 0)
 			(hide yes)
 			(show_name no)
@@
 		)
 		(property "Package" "1206 Vishay"
-			(at 35.56 137.16 0)
+			(at 33.02 138.43 0)
 			(hide yes)
 			(show_name no)
@@
 		)
 		(property "Price" "None"
-			(at 35.56 137.16 0)
+			(at 33.02 138.43 0)
 			(hide yes)
 			(show_name no)
@@
 		)
 		(property "Check_prices" "https://www.snapeda.com/parts/TEMT6000X01/Vishay/view-part/?ref=eda"
-			(at 35.56 137.16 0)
+			(at 33.02 138.43 0)
 			(hide yes)
 			(show_name no)
@@
 		)
 		(property "STANDARD" "Manufacturer Recommendations"
-			(at 35.56 137.16 0)
+			(at 33.02 138.43 0)
 			(hide yes)
 			(show_name no)
@@
 		)
 		(property "PARTREV" "1.9"
-			(at 35.56 137.16 0)
+			(at 33.02 138.43 0)
 			(hide yes)
 			(show_name no)
@@
 		)
 		(property "SnapEDA_Link" "https://www.snapeda.com/parts/TEMT6000X01/Vishay/view-part/?ref=snap"
-			(at 35.56 137.16 0)
+			(at 33.02 138.43 0)
 			(hide yes)
 			(show_name no)
@@
 		)
 		(property "MP" "TEMT6000X01"
-			(at 35.56 137.16 0)
+			(at 33.02 138.43 0)
 			(hide yes)
 			(show_name no)
@@
 		)
 		(property "Purchase-URL" "https://www.snapeda.com/api/url_track_click_mouser/?unipart_id=106092&manufacturer=Vishay Semiconductor&part_name=TEMT6000X01&search_term=temt6000x01"
-			(at 35.56 137.16 0)
+			(at 33.02 138.43 0)
 			(hide yes)
 			(show_name no)
@@
 		)
 		(property "Availability" "In Stock"
-			(at 35.56 137.16 0)
+			(at 33.02 138.43 0)
 			(hide yes)
 			(show_name no)
@@
 		)
 		(property "MANUFACTURER" "VISHAY"
-			(at 35.56 137.16 0)
+			(at 33.02 138.43 0)
 			(hide yes)
 			(show_name no)
