File: ESP32 Project/ESP32 Project.kicad_pcb (KiCad board)
At the start: 4 copper layers, 89.5 x 55 mm, 87 parts, among them J1 2338792-1, J2 B2B-PH-SM4-TB, J3 GSD090012SEU, J4 Conn_01x04_Pin, J5 Conn_01x05_Pin, Q1 TEMT6000X01, Q2 BC817, Q3 BC817, U1 MCP73871, U2 W25Q32JVSSIQ, U3 ESP32-C3-WROOM-02-H4, U4 CP2102N-Axx-xQFN20, U5 USBLC6-2SC6, U6 BME280, U7 MAX4466EXK

Commit message: some have done
Parts:
- moved J4 6.31 mm to (211.9, 62.5), turned to -90 degrees
- moved Hole 1 3.45 mm to (182.0, 86.6)
- moved Hole 2 3.43 mm to (230.1, 86.6)
Routing:
- net /Esp32-C2-02/SCL: track 0.00 -> 64.1 mm, vias 0 -> 2
- net /Esp32-C2-02/SDA: track 0.00 -> 60.9 mm, vias 0 -> 2
- net GND: track 4.29 -> 19.8 mm

Commit message: going to be end
Parts:
- moved TP5 43.8 mm to (229.6, 68.5)
- moved TP1 38.5 mm to (233.5, 89.0)
- moved TP3 35.5 mm to (238.6, 73.5)
- moved TP2 34.3 mm to (239.6, 77.5)
- moved J5 9.84 mm to (189.9, 62.5), turned to 90 degrees
- moved R22 9.24 mm to (233.3, 77.5), turned to 0 degrees
- moved TP4 8.18 mm to (263.8, 83.6)
- moved R6 7.65 mm to (186.4, 101.8)
- moved R1 7.65 mm to (188.8, 101.8)
- moved R5 7.65 mm to (184.0, 101.8)
- moved R8 7.38 mm to (191.1, 101.7)
- moved D1 7.38 mm to (193.7, 96.6)
- moved D2 7.38 mm to (191.1, 96.6)
- moved D3 7.38 mm to (196.2, 96.6)
- moved R7 7.38 mm to (193.6, 101.7)
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- renumbered PLED to D4
Connections:
- C19 pad 1: Net-(U7-IN-) -> Net-(C19-Pad1)
- R27 pad 1: Net-(U7-IN-) -> Net-(C19-Pad1)
Routing:
- net /Esp32-C2-02/GPIO18: track 0.00 -> 74.4 mm, vias 0 -> 1
- net /Esp32-C2-02/GPIO19: track 0.00 -> 72.1 mm, vias 0 -> 1
- net /Esp32-C2-02/PHOTO-C: track 0.00 -> 69.4 mm, vias 0 -> 2
- net GND: track 19.8 -> 85.6 mm, vias 12 -> 28
- net /Esp32-C2-02/GPIO8: track 0.00 -> 64.9 mm, vias 0 -> 1
- net /Esp32-C2-02/MOSI-DI: track 0.00 -> 62.7 mm
- net +3.3V: track 5.67 -> 56.7 mm, vias 5 -> 16
- net /Esp32-C2-02/MISO-DO: track 0.00 -> 45.6 mm, vias 0 -> 2
- net /Esp32-C2-02/CS: track 0.00 -> 44.8 mm, vias 0 -> 2
- net /+5Volt: track 0.00 -> 35.3 mm, vias 0 -> 1
- net /Esp32-C2-02/CS-SD: track 0.00 -> 29.0 mm
- net /Esp32-C2-02/SCLK: track 0.00 -> 25.2 mm
- net VBUS_A: track 0.00 -> 21.6 mm, vias 3 -> 5
- net /5volt usb: track 0.47 -> 14.3 mm, vias 3 -> 8
- net Net-(C24-Pad2): track 0.00 -> 12.4 mm
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- added copper zone on In1.Cu, net /5volt usb

Commit message: tomorrow is gonna be complete
Parts:
- moved S2 1.53 mm to (224.1, 108.7)
- moved S1 1.45 mm to (231.6, 108.7)
- moved C22 1.25 mm to (224.0, 106.0)
- moved C1 1.24 mm to (215.8, 101.5)
- moved R35 1.24 mm to (220.7, 107.9)
- moved C21 0.96 mm to (231.7, 106.0)
- moved C7 0.78 mm to (241.7, 67.8)
- moved Q2 0.44 mm to (224.0, 102.4), turned to -90 degrees
- moved C12 0.43 mm to (251.6, 83.5)
- moved C13 0.28 mm to (251.1, 85.8)
- moved C15 0.23 mm to (218.2, 66.0)
- moved C8 0.18 mm to (243.9, 67.2)
- turned R27 to 180 degrees
Routing:
- net /Esp32-C2-02/EN: track 7.49 -> 94.8 mm, vias 0 -> 2
- net /Esp32-C2-02/BOOT: track 0.00 -> 61.5 mm, vias 0 -> 2
- net GND: track 85.6 -> 96.5 mm, vias 28 -> 37
- net /Esp32-C2-02/SDA: track 59.6 -> 52.3 mm
- net +3.3V: track 56.7 -> 63.7 mm, vias 16 -> 17
- net Net-(U7-IN-): track 5.59 -> 10.6 mm
- net /Esp32-C2-02/RTS: track 0.00 -> 4.59 mm
- net /Esp32-C2-02/DTR: track 0.00 -> 3.61 mm
- net Net-(Q2-B): track 0.00 -> 2.49 mm
- net Net-(Q3-B): track 0.00 -> 2.05 mm
- net /Esp32-C2-02/MISO-DO: track 45.6 -> 46.8 mm
- net VBUS_A: track 21.6 -> 20.6 mm
- net Net-(C19-Pad1): track 2.38 -> 3.14 mm
- net Net-(J1-CC1): track 9.99 -> 9.35 mm

Commit message: pcb tomoroow is gonna be done
Parts:
- moved R20 0.15 mm to (242.5, 71.7)
Routing:
- net /Esp32-C2-02/TX-RX: track 0.00 -> 65.7 mm, vias 0 -> 2
- net /Esp32-C2-02/RX-TX: track 0.00 -> 65.2 mm, vias 0 -> 2
- net /Esp32-C2-02/MIC-OUT: track 8.83 -> 56.8 mm, vias 2 -> 3
- net /Esp32-C2-02/RTS: track 4.59 -> 28.4 mm, vias 0 -> 2
- net /Esp32-C2-02/DTR: track 3.61 -> 27.1 mm, vias 0 -> 2
- net GND: track 96.5 -> 104.7 mm, vias 37 -> 43
- net /Esp32-C2-02/GPIO8: track 64.9 -> 59.7 mm, vias 1 -> 2
- net +3.3V: track 63.7 -> 68.7 mm, vias 17 -> 21
- net /Esp32-C2-02/SDA: track 52.3 -> 49.6 mm
- net /Esp32-C2-02/GPIO19: track 72.1 -> 70.1 mm, vias 1 -> 2
- net /5volt usb: track 14.2 -> 16.0 mm, vias 8 -> 9
- net Net-(U4-~{RXT}/GPIO.3): track 3.47 -> 4.09 mm
- net /Esp32-C2-02/GPIO18: track 74.4 -> 74.1 mm, vias 1 -> 2
- added copper zone on In2.Cu, net +3.3V
- added copper zone on In2.Cu, net /5volt usb
- added copper zone on In1.Cu, net GND
- added copper zone on In2.Cu, net VBUS_A
- removed copper zone on In1.Cu, net +3.3V
- removed copper zone on In1.Cu, net /+5Volt
- removed copper zone on In1.Cu, net /5volt usb
- removed copper zone on In2.Cu, net GND
- removed copper zone on In1.Cu, net VBUS_A

Commit message: Agri node has comes to life!
Parts:
- added G***: LOGO, LOGO, F.Cu at (229.4, 93.7)
- added REF**: KiCad-Logo2_8mm_SilkScreen, Symbol:KiCad-Logo2_8mm_SilkScreen, F.Cu at (188.4, 69.2)
- moved R16 0.93 mm to (242.6, 84.7), turned to -90 degrees
- moved C9 0.75 mm to (218.1, 93.6)
- moved C10 0.08 mm to (215.8, 94.0)
Routing:
- net VBUS_A: track 20.6 -> 40.8 mm
- net GND: track 104.7 -> 112.7 mm, vias 43 -> 50
- net +3.3V: track 68.7 -> 67.0 mm
- net Net-(J3-DAT0): track 3.86 -> 2.29 mm
Other:
- board text added: "+3.3v"
- board text added: "2"
- board text added: "3"
- board text added: "4"
- board text added: "GND"
- board text added: "SCL"
- board text added: "SDA"
- board text added: "Tashfeen_electronics"
